Commit message: preparation for multi robot simulation

File: urdf/axis_camera_gazebo.xacro (robot description, xacro)
@@ -119,26 +119,7 @@
         <origin xyz="0.0 0.0 0.0" rpy="3.1415 0.0 0.0"/>
     </joint>
-    <ros2_control name="GazeboSimSystem" type="system">
-    <hardware>
-        <plugin>gz_ros2_control/GazeboSimSystem</plugin>
-    </hardware>
-    <joint name="pan_joint">
-      <command_interface name="position" />
-      <command_interface name="velocity" />
-      <state_interface name="position"/>
-    </joint>
-    <joint name="tilt_joint">
-      <command_interface name="position" />
-      <command_interface name="velocity" />
-      <state_interface name="position"/>
-    </joint>
-    </ros2_control>
-    <gazebo>
-      <plugin filename="gz_ros2_control-system" name="gz_ros2_control::GazeboSimROS2ControlPlugin">
-        <robot_param>robot_description</robot_param>
-        <robot_param_node>robot_state_publisher</robot_param_node>
-        <parameters>$(find ptz_gz_sim)/config/controller_params.yaml</parameters>
-      </plugin>
-    </gazebo>
+    <!-- Import ros2_control configuration -->
+    <xacro:include filename="ptz.ros2_control.xacro" />
+    <xacro:ptz_ros2_control name="MockSystem" />
     <gazebo reference="axis_camera_optical">
     <sensor name="ptz_camera" type="camera">
@@ -161,6 +142,7 @@
       <always_on>1</always_on>
       <update_rate>30</update_rate>
-      <!-- CameraZoomPlugin Configuration -->
-      <plugin name="gz::sim::systems::CameraZoomPlugin" filename="libCameraZoomPlugin.so">
+      <!-- CameraZoomPlugin Configuration - COMMENTED OUT FOR NOW -->
+      <!--
+      <plugin name="CameraZoomPlugin" filename="CameraZoomPlugin">
         <max_zoom>125.0</max_zoom>
         <slew_rate>0.425</slew_rate>
@@ -168,4 +150,5 @@
         <fb_topic>ptz_zoom_fb</fb_topic>
       </plugin>
+      -->
     </sensor>
   </gazebo>

Commit message: multi robot working + zoom working

File: urdf/axis_camera_gazebo.xacro (robot description, xacro)
@@ -82,4 +82,14 @@
             <inertia ixx="1.0" ixy="0.0" ixz="0.0" iyy="1.0" iyz="0.0" izz="1.0"/>
         </inertial>
+        <!-- ADDED: Visual for pan_link to see PTZ movement -->
+        <visual>
+            <origin xyz="0 0 0.02" rpy="0 0 0"/>
+            <geometry>
+                <box size="0.1 0.1 0.04"/>
+            </geometry>
+            <material name="Red">
+                <color rgba="1.0 0 0 0.8"/>
+            </material>
+        </visual>
     </link>
     <joint name="tilt_joint" type="revolute">
@@ -96,4 +106,14 @@
             <inertia ixx="1.0" ixy="0.0" ixz="0.0" iyy="1.0" iyz="0.0" izz="1.0"/>
         </inertial>
+        <!-- ADDED: Visual for tilt_link to see PTZ tilt movement -->
+        <visual>
+            <origin xyz="0 0 0.03" rpy="0 0 0"/>
+            <geometry>
+                <cylinder radius="0.04" length="0.06"/>
+            </geometry>
+            <material name="Green">
+                <color rgba="0 1.0 0 0.8"/>
+            </material>
+        </visual>
     </link>
     <gazebo reference="pan_joint">
@@ -113,4 +133,14 @@
             <inertia ixx="1.0" ixy="0.0" ixz="0.0" iyy="1.0" iyz="0.0" izz="1.0"/>
         </inertial>
+        <!-- ADDED: Visual for camera optical frame -->
+        <visual>
+            <origin xyz="0 0 0.01" rpy="0 0 0"/>
+            <geometry>
+                <box size="0.06 0.04 0.02"/>
+            </geometry>
+            <material name="Yellow">
+                <color rgba="1.0 1.0 0 0.9"/>
+            </material>
+        </visual>
     </link>
     <joint name="axis_camera_optical_joint" type="fixed">
@@ -119,7 +149,5 @@
         <origin xyz="0.0 0.0 0.0" rpy="3.1415 0.0 0.0"/>
     </joint>
-    <!-- Import ros2_control configuration -->
-    <xacro:include filename="ptz.ros2_control.xacro" />
-    <xacro:ptz_ros2_control name="MockSystem" />
+    <!-- Camera sensor on axis_camera_optical (original configuration) -->
     <gazebo reference="axis_camera_optical">
     <sensor name="ptz_camera" type="camera">
@@ -141,15 +169,38 @@
       </camera>
       <always_on>1</always_on>
-      <update_rate>30</update_rate>
-      <!-- CameraZoomPlugin Configuration - COMMENTED OUT FOR NOW -->
-      <!--
-      <plugin name="CameraZoomPlugin" filename="CameraZoomPlugin">
-        <max_zoom>125.0</max_zoom>
-        <slew_rate>0.425</slew_rate>
-        <topic>ptz_zoom_cmd</topic>
-        <fb_topic>ptz_zoom_fb</fb_topic>
+      <update_rate>25</update_rate>
+      <visualize>true</visualize>
+      <!-- Zoom control plugin - with retry mechanism for timing -->
+      <plugin filename="CameraZoomPlugin"
+            name="CameraZoomPlugin">
+        <max_zoom>125</max_zoom>
+        <slew_rate>5.0</slew_rate>
+        <topic>/ptz_zoom_cmd</topic>
+        <fb_topic>/ptz_zoom_fb</fb_topic>
       </plugin>
-      -->
     </sensor>
   </gazebo>
+  <!-- PTZ Joint Controllers for Gazebo Garden -->
+  <gazebo>
+    <plugin
+        filename="gz-sim-joint-position-controller-system"
+        name="gz::sim::systems::JointPositionController">
+        <joint_name>pan_joint</joint_name>
+        <topic>/pan_cmd</topic>
+        <p_gain>10</p_gain>
+        <i_gain>0.1</i_gain>
+        <d_gain>0.01</d_gain>
+    </plugin>
+  </gazebo>
+  <gazebo>
+    <plugin
+        filename="gz-sim-joint-position-controller-system"
+        name="gz::sim::systems::JointPositionController">
+        <joint_name>tilt_joint</joint_name>
+        <topic>/tilt_cmd</topic>
+        <p_gain>10</p_gain>
+        <i_gain>0.1</i_gain>
+        <d_gain>0.01</d_gain>
+    </plugin>
+  </gazebo>
 </robot>

File: urdf/ptz.ros2_control.xacro (robot description, xacro)
@@ -4,5 +4,5 @@
         <ros2_control name="${name}" type="system">
             <hardware>
-                <!-- Use mock_components instead of gz_ros2_control to avoid Gazebo plugin issues -->
+                <!-- Back to mock_components - gz_ros2_control not available -->
                 <plugin>mock_components/GenericSystem</plugin>
             </hardware>
